File: AlarmSystem/KiCad/Board/Board.kicad_pcb (KiCad board)
At the start: 2 copper layers, 3 parts, among them Q1 AO3400A

Commit message: Updated on Friday May 23rd 2025
Parts:
- moved Q1 14.4 mm to (113.1, 97.7)
- moved Q1 13.6 mm to (113.4, 84.9)
Changed lines of the file:
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@@
   (net 3 "unconnected-(Q1-D-Pad3)")
   (footprint "Package_TO_SOT_SMD:SOT-23" (layer "F.Cu")
-    (at 100.2815 88.773 180)
+    (at 113.3625 84.902 180)
     (descr "SOT, 3 Pin (https://www.jedec.org/system/files/docs/to-236h.pdf variant AB), generated with kicad-footprint-generator ipc_gullwing_generator.py")
     (tags "SOT TO_SOT_SMD")
@@
   )
   (footprint "Package_TO_SOT_SMD:SOT-23" (layer "F.Cu")
-    (at 100.33 91.059 180)
+    (at 113.133984 97.691055 180)
     (descr "SOT, 3 Pin (https://www.jedec.org/system/files/docs/to-236h.pdf variant AB), generated with kicad-footprint-generator ipc_gullwing_generator.py")
     (tags "SOT TO_SOT_SMD")
